File: Electronic/Power_Board/Power_Board.kicad_sch (KiCad schematic)
At the start: 3 parts

Commit message: Started the schematic of the power board
Parts:
- removed U?: Teensy4.1, teensy:Teensy41, symbol teensy:Teensy4.1
- removed U?: MEGA_PRO_EMBED_CH340G_/_ATMEGA2560, Mega pro:MODULE_MEGA_PRO_EMBED_CH340G___ATMEGA2560, symbol MEGA_PRO_EMBED_CH340G___ATMEGA2560:MEGA_PRO_EMBED_CH340G_/_ATMEGA2560
- removed U?: RASPBERRYPI4_4GB, Raspberry:MODULE_RASPBERRYPI4_4GB, symbol RASPBERRYPI4_4GB:RASPBERRYPI4_4GB
- added C? (x3): 4.7u, symbol Device:C
- added J?: Conn_02x10_Counter_Clockwise, symbol Connector_Generic:Conn_02x10_Counter_Clockwise
- added PS1, PS?: TEN_50-2413, Traco:CONV_TEN_50-2413, symbol TEN_50-2413:TEN_50-2413
- added PS?: TEN_30-2411, Traco:CONV_TEN_50-2413, symbol TEN_50-2413:TEN_50-2413
- added R?: 0, symbol Device:R
Connections:
- new net +BATT: C?.1, C?.1, C?.1, J?.13 (Pin_13), J?.14 (Pin_14), J?.15 (Pin_15), J?.16 (Pin_16), J?.17 (Pin_17), J?.18 (Pin_18), J?.19 (Pin_19), J?.20 (Pin_20), PS1.1 (+VIN(VCC)), PS?.1 (+VIN(VCC)), PS?.1 (+VIN(VCC))
- new net -BATT: C?.2, C?.2, C?.2, J?.10 (Pin_10), J?.11 (Pin_11), J?.12 (Pin_12), J?.5 (Pin_5), J?.6 (Pin_6), J?.7 (Pin_7), J?.8 (Pin_8), J?.9 (Pin_9), PS1.2 (-VIN(GND)), PS?.2 (-VIN(GND)), PS?.2 (-VIN(GND))
- new net 5V ON/OFF: PS?.3 (ON/OFF), R?.2
- new net 5V ON/OFF connector: J?.3 (Pin_3), R?.1
- new net GND: J?.4 (Pin_4)
- new net Prop ON/OFF: J?.2 (Pin_2), PS1.3 (ON/OFF), PS?.3 (ON/OFF)
- new net TDK ON/OFF: J?.1 (Pin_1)

Commit message: Added documentation and more work on KiCad
Parts:
- added J2: Conn_02x10_Counter_Clockwise, Connector_PinSocket_2.54mm:PinSocket_2x20_P2.54mm_Vertical_SMD, symbol Connector_Generic:Conn_02x10_Counter_Clockwise
- added PS2: I6A24014A033V-001-R, TDK converter:CONV_I6A24014A033V-001-R, symbol I6A24014A033V-001-R:I6A24014A033V-001-R
- added R2, R3: 0, Resistor_SMD:R_0201_0603Metric_Pad0.64x0.40mm_HandSolder, symbol Device:R
- added U1: TB67H400AFTG_EL, Toshiba:TB67H400AFTG_EL, symbol Toshiba TB67H400:TB67H400AFTG_EL
- C1, C2, C3: renamed from C?; footprint (none) -> Capacitor_THT:CP_Radial_D12.5mm_P7.50mm
- J1: renamed from J?; footprint (none) -> Connector_PinSocket_2.54mm:PinSocket_2x20_P2.54mm_Vertical_SMD
- R1: renamed from R?; footprint (none) -> Resistor_SMD:R_0201_0603Metric_Pad0.64x0.40mm_HandSolder
- gave numbers to parts that had none: 2
Connections:
- net +BATT: now also PS2.1 (VIN(+))
- net -BATT: now also PS2.3 (VIN(-))
- net GND: now also PS1.5 (-VOUT), PS3.5 (-VOUT), PS4.5 (-VOUT), J2.10 (Pin_10), J2.11 (Pin_11), J2.12 (Pin_12), J2.5 (Pin_5), J2.6 (Pin_6), J2.7 (Pin_7), J2.8 (Pin_8), J2.9 (Pin_9)
- net Prop ON/OFF: now also R2.2; no longer J1.2 (Pin_2)
- net TDK ON/OFF: now also R3.2; no longer J1.1 (Pin_1)
- net Prop_1 out: now reaches PS1.4 (+VOUT)
- net Prop_1 out: now also J2.1 (Pin_1), J2.2 (Pin_2), J2.3 (Pin_3), J2.4 (Pin_4)
- net 5V out: now reaches PS4.4 (+VOUT)
- net 5V out: now also J2.13 (Pin_13), J2.14 (Pin_14), J2.15 (Pin_15), J2.16 (Pin_16)
- net Prop_2 out: now reaches PS3.4 (+VOUT)
- net Prop_2 out: now also J2.17 (Pin_17), J2.18 (Pin_18), J2.19 (Pin_19), J2.20 (Pin_20)
- new net Prop ON/OFF connector: J1.2 (Pin_2), R3.1
- new net TDK ON/OFF connector: J1.1 (Pin_1), R2.1
Other:
- note added: "I made a mistake last year, need to check IRL PCB"
- note added: "On: 3.5 to 12 VDC or open circuit Off: 0 to 1.2 VDC or short circuit Refers to 'Remote' and '-Vin' Pin"
- moved on the sheet: R1

Commit message: More KiCad
Parts:
- removed J1: Conn_02x10_Counter_Clockwise, Connector_PinSocket_2.54mm:PinSocket_2x20_P2.54mm_Vertical_SMD, symbol Connector_Generic:Conn_02x10_Counter_Clockwise
- added J?: Conn_02x20_Counter_Clockwise, Connector_PinSocket_2.54mm:PinSocket_2x20_P2.54mm_Vertical_SMD, symbol Connector_Generic:Conn_02x20_Counter_Clockwise
- J?: renamed from J2; footprint Connector_PinSocket_2.54mm:PinSocket_2x20_P2.54mm_Vertical_SMD -> Connector_PinSocket_2.54mm:PinSocket_2x10_P2.54mm_Vertical_SMD
- R?: renamed from R2; footprint Resistor_SMD:R_0201_0603Metric_Pad0.64x0.40mm_HandSolder -> Jumper:SolderJumper-2_P1.3mm_Open_Pad1.0x1.5mm
- R?: renamed from R3; footprint Resistor_SMD:R_0201_0603Metric_Pad0.64x0.40mm_HandSolder -> Jumper:SolderJumper-2_P1.3mm_Open_Pad1.0x1.5mm
- R?: renamed from R1; footprint Resistor_SMD:R_0201_0603Metric_Pad0.64x0.40mm_HandSolder -> Jumper:SolderJumper-2_P1.3mm_Open_RoundedPad1.0x1.5mm
- renumbered C1 to C?, C3 to C?, C2 to C?, PS1 to PS?, PS2 to PS?, PS4 to PS?, PS3 to PS?, U1 to U?
Connections:
- net +BATT: now also J?.27 (Pin_27), J?.28 (Pin_28), J?.29 (Pin_29), J?.30 (Pin_30), J?.31 (Pin_31), J?.32 (Pin_32), J?.33 (Pin_33), J?.34 (Pin_34), J?.35 (Pin_35), J?.36 (Pin_36)
- net -BATT: now also J?.15 (Pin_15), J?.16 (Pin_16), J?.17 (Pin_17), J?.18 (Pin_18), J?.19 (Pin_19), J?.20 (Pin_20), J?.21 (Pin_21), J?.22 (Pin_22), J?.23 (Pin_23), J?.24 (Pin_24), J?.25 (Pin_25), J?.26 (Pin_26)
- net 5V ON/OFF connector: now also J?.13 (Pin_13)
- net GND: now also J?.14 (Pin_14)
- net Prop ON/OFF connector: now also J?.12 (Pin_12)
- net TDK ON/OFF connector: now also J?.11 (Pin_11), J?.8 (Pin_8)
- new net PWM_Motor_1: J?.10 (Pin_10)
- new net PWM_Motor_2: J?.9 (Pin_9)
Other:
- moved on the sheet: C?, PS?, R?
